File: hardware/aquabox_final/rtc_sd.kicad_sch (KiCad schematic)
At the start: 0 parts

Commit message: Implementação do RTC
Parts:
- added BT1: Battery_Cell, Battery:Battery_Panasonic_CR2032-HFN_Horizontal_CircularHoles, symbol Device:Battery_Cell
- added C9: 100n, symbol Device:C
- added R46, R47, R48: 4K7, symbol Device:R
- added U14: DS3231M, Package_SO:SOIC-16W_7.5x10.3mm_P1.27mm, symbol Timer_RTC:DS3231M
Connections:
- new net: R48.2, U14.3 (~{INT}/SQW)
- new net: BT1.1 (+), C9.1, U14.14 (VBAT)
- new net +3.3V: R46.1, R47.1, R48.1, U14.2 (VCC)
- new net GND: BT1.2 (-), C9.2, U14.10 (GND), U14.11 (GND), U14.12 (GND), U14.13 (GND), U14.5 (GND), U14.6 (GND), U14.7 (GND), U14.8 (GND), U14.9 (GND)
- new net I2C_SCL: R47.2, U14.16 (SCL)
- new net I2C_SDA: R46.2, U14.15 (SDA)
- no-connect marks 0 -> 2
