File: hardware/aquabox_final/rtc_sd.kicad_sch (KiCad schematic)
At the start: 6 parts, among them U14 DS3231M

Commit message: Atualização
Connections:
- net I2C_SCL: now also R46.2; no longer R47.2
- net I2C_SDA: now also R47.2; no longer R46.2
Changed lines of the file:
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@@
+	)
+	(junction
+		(at 121.92 90.17)
+		(diameter 0)
+		(color 0 0 0 0)
 	)
 	(junction
@@
 	)
 	(junction
-		(at 130.81 90.17)
-		(diameter 0)
-		(color 0 0 0 0)
-	)
-	(junction
 		(at 130.81 71.12)
 		(diameter 0)
@@
 	)
 	(junction
-		(at 121.92 92.71)
+		(at 130.81 92.71)
 		(diameter 0)
 		(color 0 0 0 0)
@@
 	(wire
 		(pts
-			(xy 130.81 81.28) (xy 130.81 90.17)
-		)
-		(stroke
-			(width 0)
-			(type default)
-		)
-	)
-	(wire
-		(pts
-			(xy 121.92 92.71) (xy 137.16 92.71)
-		)
-		(stroke
-			(width 0)
-			(type default)
-		)
-	)
-	(wire
-		(pts
 			(xy 173.99 82.55) (xy 173.99 93.98)
 		)
@@
 	(wire
 		(pts
-			(xy 121.92 81.28) (xy 121.92 92.71)
-		)
-		(stroke
-			(width 0)
-			(type default)
-		)
-	)
-	(wire
-		(pts
-			(xy 130.81 90.17) (xy 137.16 90.17)
+			(xy 130.81 92.71) (xy 137.16 92.71)
 		)
 		(stroke
@@
 	(wire
 		(pts
+			(xy 107.95 92.71) (xy 130.81 92.71)
+		)
+		(stroke
+			(width 0)
+			(type default)
+		)
+	)
+	(wire
+		(pts
+			(xy 107.95 90.17) (xy 121.92 90.17)
+		)
+		(stroke
+			(width 0)
+			(type default)
+		)
+	)
+	(wire
+		(pts
 			(xy 130.81 71.12) (xy 130.81 73.66)
 		)
@@
 	(wire
 		(pts
-			(xy 102.87 92.71) (xy 121.92 92.71)
-		)
-		(stroke
-			(width 0)
-			(type default)
-		)
-	)
-	(wire
-		(pts
 			(xy 149.86 85.09) (xy 149.86 82.55)
 		)
@@
 	(wire
 		(pts
+			(xy 121.92 81.28) (xy 121.92 90.17)
+		)
+		(stroke
+			(width 0)
+			(type default)
+		)
+	)
+	(wire
+		(pts
+			(xy 121.92 90.17) (xy 137.16 90.17)
+		)
+		(stroke
+			(width 0)
+			(type default)
+		)
+	)
+	(wire
+		(pts
 			(xy 165.1 71.12) (xy 165.1 73.66)
 		)
@@
 	(wire
 		(pts
-			(xy 102.87 90.17) (xy 130.81 90.17)
+			(xy 130.81 81.28) (xy 130.81 92.71)
 		)
 		(stroke
@@
 		)
 	)
-	(global_label "I2C_SDA"
+	(hierarchical_label "I2C_SDA"
 		(shape bidirectional)
-		(at 102.87 92.71 180)
-		(fields_autoplaced yes)
+		(at 107.95 92.71 180)
 		(effects
 			(font
@@
 			(justify right)
 		)
-		(property "Intersheetrefs" "${INTERSHEET_REFS}"
-			(at 91.1535 92.71 0)
-			(hide yes)
-			(show_name no)
-			(do_not_autoplace no)
-			(effects
-				(font
-					(size 1.27 1.27)
-				)
-				(justify right)
-			)
-		)
-	)
-	(global_label "I2C_SCL"
+	)
+	(hierarchical_label "I2C_SCL"
 		(shape input)
-		(at 102.87 90.17 180)
-		(fields_autoplaced yes)
+		(at 107.95 90.17 180)
 		(effects
 			(font
@@
 			(justify right)
 		)
-		(property "Intersheetrefs" "${INTERSHEET_REFS}"
-			(at 92.3253 90.17 0)
-			(hide yes)
-			(show_name no)
-			(do_not_autoplace no)
-			(effects
-				(font
-					(size 1.27 1.27)
-				)
-				(justify right)
-			)
-		)
-	)
+	)
