File: hardware/aquabox_final/power.kicad_sch (KiCad schematic)
At the start: 13 parts, among them J1 Entrada de 12V, J2 AC 220V, U1 HLK-10M05

Commit message: Atualização
Changed lines of the file:
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@@
 	)
 	(hierarchical_label "R_NO"
-		(shape output)
+		(shape input)
 		(at 80.01 105.41 0)
 		(effects
@@
 	)
 	(hierarchical_label "R_C"
-		(shape input)
+		(shape output)
 		(at 93.98 113.03 0)
 		(effects
