File: hardware/aquabox_final/inputs.kicad_sch (KiCad schematic)
At the start: 39 parts, among them J4 Sensor de Fluxo, J5 Caixa_1, J6 Caixa_2, J7 Caixa_3, U3 PC817, U4 PC817, U5 PC817, U6 PC817, U7 PC817, U8 PC817, U9 PC817

Commit message: Atualização
Connections:
- net GND1: now also J5.3 (Pin_3), J6.3 (Pin_3), J7.3 (Pin_3); no longer J5.1 (Pin_1), J6.1 (Pin_1), J7.1 (Pin_1)
- net SENSOR_H1: now also J5.2 (Pin_2); no longer J5.3 (Pin_3)
- net SENSOR_H2: now also J6.2 (Pin_2); no longer J6.3 (Pin_3)
- net SENSOR_H3: now also J7.2 (Pin_2); no longer J7.3 (Pin_3)
- net SENSOR_L1: now also J5.1 (Pin_1); no longer J5.2 (Pin_2)
- net SENSOR_L2: now also J6.1 (Pin_1); no longer J6.2 (Pin_2)
- net SENSOR_L3: now also J7.1 (Pin_1); no longer J7.2 (Pin_2)
- net T1_HIGH renamed S1_HIGH
- net T1_LOW renamed S1_LOW
- net T2_HIGH renamed S2_HIGH
- net T2_LOW renamed S2_LOW
- net T3_HIGH renamed S3_HIGH
- net T3_LOW renamed S3_LOW
Other:
- moved on the sheet: D7, J4, J5, J6, J7, R18, R21, R24, U7
