File: hardware/aquabox_final/inputs.kicad_sch (KiCad schematic)
At the start: 39 parts, among them J4 Sensor de Fluxo, J5 Caixa_1, J6 Caixa_2, J7 Caixa_3, U3 PC817, U4 PC817, U5 PC817, U6 PC817, U7 PC817, U8 PC817, U9 PC817

Commit message: Atualização
Parts:
- renumbered D8 to D7, D9 to D8, D7 to D9, J5 to J3, J6 to J4, J7 to J5, J4 to J6, R13 to R10, R14 to R11, R15 to R12, R16 to R13, R17 to R14, R19 to R15, R20 to R16, R22 to R17, R23 to R18, R25 to R19, R26 to R20, R18 to R21, R27 to R22, R28 to R23, R21 to R24, R29 to R25, R30 to R26, R24 to R27, R10 to R7, R11 to R8, R12 to R9, U7 to U10, U3 to U4, U4 to U5, U5 to U6, U6 to U7

Commit message: Esquemático Aquabox III
Parts:
- R25: renamed from R21; value 1K -> 220R
- renumbered R24 to R19, R19 to R20, R20 to R21, R27 to R24, R25 to R26, R26 to R27, U9 to U10, U10 to U8, U8 to U9
Connections:
- net +12V: no longer R25.1
- net +3.3V: now also R25.1
- net FLOW_COUNTER: now also D9.1 (K)
- net FLOW_SENSOR: no longer D9.1 (K)
Other:
- moved on the sheet: D9, R19, R24, R25, U8
