File: hardware/aquabox_final/solenoids.kicad_sch (KiCad schematic)
At the start: 33 parts, among them J8 Screw_Terminal_01x04, K1 Relay_SPDT, Q1 BC337, Q10 BC337, Q2 BC327, Q3 BC337, Q4 BC327, Q5 BC337, Q6 BC327, Q7 IRLZ44N, Q8 IRLZ44N, Q9 IRLZ44N, U10 PC817, U11 PC817, U12 PC817, U13 PC817

Commit message: Atualização
Connections:
- net R_C: now reaches K1.11
- net R_NO: now reaches K1.14
Changed lines of the file:
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@@
+	(wire
+		(pts
+			(xy 245.11 91.44) (xy 242.57 91.44)
+		)
+		(stroke
+			(width 0)
+			(type default)
+		)
+	)
 	(wire
 		(pts
@@
 	(wire
 		(pts
+			(xy 240.03 110.49) (xy 240.03 113.03)
+		)
+		(stroke
+			(width 0)
+			(type default)
+		)
+	)
+	(wire
+		(pts
 			(xy 156.21 114.3) (xy 161.29 114.3)
 		)
@@
 	(wire
 		(pts
+			(xy 242.57 91.44) (xy 242.57 95.25)
+		)
+		(stroke
+			(width 0)
+			(type default)
+		)
+	)
+	(wire
+		(pts
 			(xy 109.22 157.48) (xy 109.22 165.1)
 		)
@@
 		(pts
 			(xy 170.18 49.53) (xy 181.61 49.53)
+		)
+		(stroke
+			(width 0)
+			(type default)
+		)
+	)
+	(wire
+		(pts
+			(xy 240.03 113.03) (xy 245.11 113.03)
 		)
 		(stroke
@@
 		)
 	)
+	(hierarchical_label "R_C"
+		(shape input)
+		(at 245.11 113.03 0)
+		(effects
+			(font
+				(size 1.27 1.27)
+			)
+			(justify left)
+		)
+	)
+	(hierarchical_label "R_NO"
+		(shape output)
+		(at 245.11 91.44 0)
+		(effects
+			(font
+				(size 1.27 1.27)
+			)
+			(justify left)
+		)
+	)

Commit message: Atualização
Parts:
- renumbered J8 to J7, R31 to R28, R32 to R29, R33 to R30, R34 to R31, R35 to R32, R36 to R33, R37 to R34, R38 to R35, R39 to R36, R40 to R37, R41 to R38, R42 to R39, R43 to R40, R44 to R41, R45 to R42, U10 to U11, U11 to U12, U12 to U13, U13 to U14
Other:
- moved on the sheet: J7

Commit message: Esquemático Aquabox III
Other:
- title: Solenóides e Bomba -> Outputs
Changed lines of the file:
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@@
 	(paper "A4")
 	(title_block
-		(title "Solenóides e Bomba")
+		(title "Outputs")
 		(date "2026-06-03")
 		(rev "1.0.0")
