File: hardware/aquabox_final/Interfaces.kicad_sch (KiCad schematic)
At the start: 14 parts, among them SW1 BOMBA, SW2 MANUAL?AUTOMATICO

Commit message: Atualização
Parts:
- SW2: value MANUAL?AUTOMATICO -> MANUAL/AUTOMATICO
Other:
- moved on the sheet: C3, C4, C5, C7, R4, R5, R6, R8

Commit message: Atualização
Parts:
- added J3: Conn_01x05, symbol Connector_Generic:Conn_01x05
- added R49, R50, R51, R52, R53, R54: 10K, symbol Device:R
- added U15: 74HC14, symbol 74xx:74HC14
Connections:
- net +3.3V: now also U15.14 (VCC)
- net BOMBA_ON_OFF: now also U15.2; no longer C6.1, R7.2, SW2.2 (B)
- net BTN_BACK: now also U15.12; no longer C7.1, R8.2
- net BTN_DOWN: now also U15.8; no longer C4.1, R5.2
- net BTN_ENTER: now also U15.10; no longer C5.1, R6.2
- net BTN_UP: now also U15.6; no longer C3.1, R4.2
- net GND: now also U15.7 (GND)
- net MAN_AUTO: now also U15.4; no longer C8.1, R9.2, SW1.2 (B)
- new net: C5.1, R49.2, U15.11
- new net: C4.1, R51.2, U15.9
- new net: C8.1, R54.2, U15.3
- new net: C3.1, R52.2, U15.5
- new net: C6.1, R53.2, U15.1
- new net: J3.2 (Pin_2), R5.2, R51.1
- new net: J3.1 (Pin_1), R4.2, R52.1
- new net: J3.3 (Pin_3), R49.1, R6.2
- new net: J3.4 (Pin_4), R50.1, R8.2
- new net: R53.1, R7.2, SW2.2 (B)
- new net: C7.1, R50.2, U15.13
- new net: R54.1, R9.2, SW1.2 (B)
Other:
- moved on the sheet: C3, C4, C5, C6, C7, C8, R4, R5, R6, R8, SW1, SW2

Commit message: Atualização
Parts:
- removed SW1: BOMBA, symbol Switch:SW_SPST
- removed SW2: MANUAL/AUTOMATICO, symbol Switch:SW_SPST
- added J10: Conn_01x10, symbol Connector_Generic:Conn_01x10
- added J8: Conn_01x03, symbol Connector_Generic:Conn_01x03
- renumbered C6 to C4, C8 to C5, C3 to C6, C4 to C7, C5 to C8, C7 to C9, J3 to J9, R7 to R43, R4 to R44, R9 to R45, R5 to R46, R6 to R47, R53 to R48, R54 to R49, R8 to R50, R52 to R51, R51 to R52, R49 to R53, R50 to R54
Connections:
- net +3.3V: now also J10.2 (Pin_2)
- net GND: now also J9.5 (Pin_5), J10.10 (Pin_10), J8.3 (Pin_3)
- net SD_CS: now also J10.9 (Pin_9)
- net SPI_MOSI: now also J10.7 (Pin_7)
- net SPI_SCK: now also J10.8 (Pin_8)
- net TFT_BL: now also J10.3 (Pin_3)
- net TFT_CS: now also J10.5 (Pin_5)
- net TFT_DC: now also J10.4 (Pin_4)
- net TFT_RST: now also J10.6 (Pin_6)
- net at R43.2, R48.1: now also J8.1 (Pin_1)
- net at R45.2, R49.1: now also J8.2 (Pin_2)
- new net +5V: J10.1 (Pin_1)
Other:
- note added: "BACK"
- note added: "BOMBA"
- note added: "DOWN"
- note added: "ENTER"
- note added: "MANUAL/AUTO"
- note added: "UP"
- moved on the sheet: C4, C5, C6, C7, C8, C9, J9, R43, R44, R45, R46, R47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

Commit message: Atualização
Parts:
- added C10: 100n, symbol Device:C
Connections:
- net +3.3V: now also C10.1
- net GND: now also C10.2
Changed lines of the file:
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@@
 	)
 	(junction
+		(at 73.66 147.32)
+		(diameter 0)
+		(color 0 0 0 0)
+	)
+	(junction
 		(at 80.01 107.95)
 		(diameter 0)
@@
 		(color 0 0 0 0)
 	)
+	(junction
+		(at 73.66 175.26)
+		(diameter 0)
+		(color 0 0 0 0)
+	)
 	(wire
 		(pts
@@
 	(wire
 		(pts
+			(xy 82.55 175.26) (xy 73.66 175.26)
+		)
+		(stroke
+			(width 0)
+			(type default)
+		)
+	)
+	(wire
+		(pts
 			(xy 64.77 88.9) (xy 72.39 88.9)
 		)
@@
 	(wire
 		(pts
+			(xy 82.55 147.32) (xy 73.66 147.32)
+		)
+		(stroke
+			(width 0)
+			(type default)
+		)
+	)
+	(wire
+		(pts
 			(xy 109.22 125.73) (xy 146.05 125.73)
 		)
@@
 	(wire
 		(pts
-			(xy 73.66 173.99) (xy 73.66 177.8)
+			(xy 73.66 173.99) (xy 73.66 175.26)
 		)
 		(stroke
@@
 	(wire
 		(pts
+			(xy 82.55 157.48) (xy 82.55 147.32)
+		)
+		(stroke
+			(width 0)
+			(type default)
+		)
+	)
+	(wire
+		(pts
 			(xy 64.77 100.33) (xy 64.77 102.87)
 		)
@@
 	(wire
 		(pts
-			(xy 73.66 144.78) (xy 73.66 148.59)
+			(xy 73.66 144.78) (xy 73.66 147.32)
 		)
 		(stroke
@@
 	(wire
 		(pts
+			(xy 73.66 147.32) (xy 73.66 148.59)
+		)
+		(stroke
+			(width 0)
+			(type default)
+		)
+	)
+	(wire
+		(pts
 			(xy 59.69 43.18) (xy 59.69 45.72)
 		)
@@
 	(wire
 		(pts
+			(xy 82.55 165.1) (xy 82.55 175.26)
+		)
+		(stroke
+			(width 0)
+			(type default)
+		)
+	)
+	(wire
+		(pts
 			(xy 231.14 71.12) (xy 234.95 71.12)
 		)
@@
 	(wire
 		(pts
+			(xy 73.66 175.26) (xy 73.66 177.8)
+		)
+		(stroke
+			(width 0)
+			(type default)
+		)
+	)
+	(wire
+		(pts
 			(xy 226.06 68.58) (xy 234.95 68.58)
 		)
@@
 	(symbol
 		(lib_id "Device:C")
+		(at 82.55 161.29 0)
+		(unit 1)
+		(body_style 1)
+		(exclude_from_sim no)
+		(in_bom yes)
+		(on_board yes)
+		(in_pos_files yes)
+		(dnp no)
+		(fields_autoplaced yes)
+		(property "Reference" "C10"
+			(at 86.36 160.0199 0)
+			(show_name no)
+			(do_not_autoplace no)
+			(effects
+				(font
+					(size 1.27 1.27)
+				)
+				(justify left)
+			)
+		)
+		(property "Value" "100n"
+			(at 86.36 162.5599 0)
+			(show_name no)
+			(do_not_autoplace no)
+			(effects
+				(font
+					(size 1.27 1.27)
+				)
+				(justify left)
+			)
+		)
+		(property "Footprint" ""
+			(at 83.5152 165.1 0)
+			(hide yes)
+			(show_name no)
+			(do_not_autoplace no)
+			(effects
+				(font
+					(size 1.27 1.27)
+				)
+			)
+		)
+		(property "Datasheet" ""
+			(at 82.55 161.29 0)
+			(hide yes)
+			(show_name no)
+			(do_not_autoplace no)
+			(effects
+				(font
+					(size 1.27 1.27)
+				)
+			)
+		)
+		(property "Description" "Unpolarized capacitor"
+			(at 82.55 161.29 0)
+			(hide yes)
+			(show_name no)
+			(do_not_autoplace no)
+			(effects
+				(font
+					(size 1.27 1.27)
+				)
+			)
+		)
+		(pin "2"
+		)
+		(pin "1"
+		)
+		(instances
+			(project "aquabox_final"
+				(path "/c895ac8d-c639-4fea-ba83-739985d9c75e/6a1a24a6-7a05-4323-8d4e-6696d3969bdc"
+					(reference "C10")
+					(unit 1)
+				)
+			)
+		)
+	)
+	(symbol
+		(lib_id "Device:C")
 		(at 111.76 140.97 0)
 		(unit 1)
@@
 		(in_pos_files yes)
 		(dnp no)
-		(fields_autoplaced yes)
 		(property "Reference" "U15"
-			(at 80.01 160.0199 0)
+			(at 60.452 159.004 0)
 			(show_name no)
 			(do_not_autoplace no)
@@
 		)
 		(property "Value" "74HC14"
-			(at 80.01 162.5599 0)
+			(at 60.452 161.544 0)
 			(show_name no)
 			(do_not_autoplace no)

Commit message: Atualização
Parts:
- renumbered C8 to C10, C9 to C11, C10 to C5, C4 to C6, C5 to C7, C6 to C8, C7 to C9
Changed lines of the file:
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@@
 		(dnp no)
 		(fields_autoplaced yes)
-		(property "Reference" "C8"
+		(property "Reference" "C10"
 			(at 138.43 139.6999 0)
 			(show_name no)
@@
 			(project "aquabox_final"
 				(path "/c895ac8d-c639-4fea-ba83-739985d9c75e/6a1a24a6-7a05-4323-8d4e-6696d3969bdc"
-					(reference "C8")
+					(reference "C10")
 					(unit 1)
 				)
@@
 		(dnp no)
 		(fields_autoplaced yes)
-		(property "Reference" "#PWR063"
+		(property "Reference" "#PWR065"
 			(at 54.61 66.04 0)
 			(hide yes)
@@
 			(project "aquabox_final"
 				(path "/c895ac8d-c639-4fea-ba83-739985d9c75e/6a1a24a6-7a05-4323-8d4e-6696d3969bdc"
-					(reference "#PWR063")
+					(reference "#PWR065")
 					(unit 1)
 				)
@@
 		(dnp no)
 		(fields_autoplaced yes)
-		(property "Reference" "C7"
+		(property "Reference" "C9"
 			(at 127 139.6999 0)
 			(show_name no)
@@
 			(project "aquabox_final"
 				(path "/c895ac8d-c639-4fea-ba83-739985d9c75e/6a1a24a6-7a05-4323-8d4e-6696d3969bdc"
-					(reference "C7")
+					(reference "C9")
 					(unit 1)
 				)
@@
 		(dnp no)
 		(fields_autoplaced yes)
-		(property "Reference" "#PWR073"
+		(property "Reference" "#PWR075"
 			(at 231.14 81.28 0)
 			(hide yes)
@@
 			(project "aquabox_final"
 				(path "/c895ac8d-c639-4fea-ba83-739985d9c75e/6a1a24a6-7a05-4323-8d4e-6696d3969bdc"
-					(reference "#PWR073")
+					(reference "#PWR075")
 					(unit 1)
 				)
@@
 		(dnp no)
 		(fields_autoplaced yes)
-		(property "Reference" "#PWR071"
+		(property "Reference" "#PWR073"
 			(at 222.25 46.99 0)
 			(hide yes)
@@
 			(project "aquabox_final"
 				(path "/c895ac8d-c639-4fea-ba83-739985d9c75e/6a1a24a6-7a05-4323-8d4e-6696d3969bdc"
-					(reference "#PWR071")
+					(reference "#PWR073")
 					(unit 1)
 				)
@@
 		(dnp no)
 		(fields_autoplaced yes)
-		(property "Reference" "C10"
+		(property "Reference" "C5"
 			(at 86.36 160.0199 0)
 			(show_name no)
@@
 			(project "aquabox_final"
 				(path "/c895ac8d-c639-4fea-ba83-739985d9c75e/6a1a24a6-7a05-4323-8d4e-6696d3969bdc"
-					(reference "C10")
+					(reference "C5")
 					(unit 1)
 				)
@@
 		(dnp no)
 		(fields_autoplaced yes)
-		(property "Reference" "C6"
+		(property "Reference" "C8"
 			(at 115.57 139.6999 0)
 			(show_name no)
@@
 			(project "aquabox_final"
 				(path "/c895ac8d-c639-4fea-ba83-739985d9c75e/6a1a24a6-7a05-4323-8d4e-6696d3969bdc"
-					(reference "C6")
+					(reference "C8")
 					(unit 1)
 				)
@@
 		(dnp no)
 		(fields_autoplaced yes)
-		(property "Reference" "#PWR069"
+		(property "Reference" "#PWR071"
 			(at 106.68 78.74 0)
 			(hide yes)
@@
 			(project "aquabox_final"
 				(path "/c895ac8d-c639-4fea-ba83-739985d9c75e/6a1a24a6-7a05-4323-8d4e-6696d3969bdc"
-					(reference "#PWR069")
+					(reference "#PWR071")
 					(unit 1)
 				)
@@
 		(dnp no)
 		(fields_autoplaced yes)
-		(property "Reference" "C4"
+		(property "Reference" "C6"
 			(at 97.79 63.4999 0)
 			(show_name no)
@@
 			(project "aquabox_final"
 				(path "/c895ac8d-c639-4fea-ba83-739985d9c75e/6a1a24a6-7a05-4323-8d4e-6696d3969bdc"
-					(reference "C4")
+					(reference "C6")
 					(unit 1)
 				)
@@
 		(dnp no)
 		(fields_autoplaced yes)
-		(property "Reference" "#PWR064"
+		(property "Reference" "#PWR066"
 			(at 58.42 125.73 0)
 			(hide yes)
@@
 			(project "aquabox_final"
 				(path "/c895ac8d-c639-4fea-ba83-739985d9c75e/6a1a24a6-7a05-4323-8d4e-6696d3969bdc"
-					(reference "#PWR064")
+					(reference "#PWR066")
 					(unit 1)
 				)
@@
 		(dnp no)
 		(fields_autoplaced yes)
-		(property "Reference" "#PWR070"
+		(property "Reference" "#PWR072"
 			(at 146.05 158.75 0)
 			(hide yes)
@@
 			(project "aquabox_final"
 				(path "/c895ac8d-c639-4fea-ba83-739985d9c75e/6a1a24a6-7a05-4323-8d4e-6696d3969bdc"
-					(reference "#PWR070")
+					(reference "#PWR072")
 					(unit 1)
 				)
@@
 		(dnp no)
 		(fields_autoplaced yes)
-		(property "Reference" "#PWR072"
+		(property "Reference" "#PWR074"
 			(at 229.87 46.99 0)
 			(hide yes)
@@
 			(project "aquabox_final"
 				(path "/c895ac8d-c639-4fea-ba83-739985d9c75e/6a1a24a6-7a05-4323-8d4e-6696d3969bdc"
-					(reference "#PWR072")
+					(reference "#PWR074")
 					(unit 1)
 				)
@@
 		(dnp no)
 		(fields_autoplaced yes)
-		(property "Reference" "#PWR065"
+		(property "Reference" "#PWR067"
 			(at 72.39 33.02 0)
 			(hide yes)
@@
 			(project "aquabox_final"
 				(path "/c895ac8d-c639-4fea-ba83-739985d9c75e/6a1a24a6-7a05-4323-8d4e-6696d3969bdc"
-					(reference "#PWR065")
+					(reference "#PWR067")
 					(unit 1)
 				)
@@
 		(dnp no)
 		(fields_autoplaced yes)
-		(property "Reference" "#PWR068"
+		(property "Reference" "#PWR070"
 			(at 87.63 90.17 0)
 			(hide yes)
@@
 			(project "aquabox_final"
 				(path "/c895ac8d-c639-4fea-ba83-739985d9c75e/6a1a24a6-7a05-4323-8d4e-6696d3969bdc"
-					(reference "#PWR068")
+					(reference "#PWR070")
 					(unit 1)
 				)
@@
 		(dnp no)
 		(fields_autoplaced yes)
-		(property "Reference" "#PWR066"
+		(property "Reference" "#PWR068"
 			(at 73.66 148.59 0)
 			(hide yes)
@@
 			(project "aquabox_final"
 				(path "/c895ac8d-c639-4fea-ba83-739985d9c75e/6a1a24a6-7a05-4323-8d4e-6696d3969bdc"
-					(reference "#PWR066")
+					(reference "#PWR068")
 					(unit 1)
 				)
@@
 		(dnp no)
 		(fields_autoplaced yes)
-		(property "Reference" "#PWR067"
+		(property "Reference" "#PWR069"
 			(at 73.66 184.15 0)
 			(hide yes)
@@
 			(project "aquabox_final"
 				(path "/c895ac8d-c639-4fea-ba83-739985d9c75e/6a1a24a6-7a05-4323-8d4e-6696d3969bdc"
-					(reference "#PWR067")
+					(reference "#PWR069")
 					(unit 1)
 				)
@@
 		(dnp no)
 		(fields_autoplaced yes)
-		(property "Reference" "C5"
+		(property "Reference" "C7"
 			(at 110.49 63.4999 0)
 			(show_name no)
@@
 			(project "aquabox_final"
 				(path "/c895ac8d-c639-4fea-ba83-739985d9c75e/6a1a24a6-7a05-4323-8d4e-6696d3969bdc"
-					(reference "C5")
+					(reference "C7")
 					(unit 1)
 				)
@@
 		(dnp no)
 		(fields_autoplaced yes)
-		(property "Reference" "C9"
+		(property "Reference" "C11"
 			(at 149.86 139.6999 0)
 			(show_name no)
@@
 			(project "aquabox_final"
 				(path "/c895ac8d-c639-4fea-ba83-739985d9c75e/6a1a24a6-7a05-4323-8d4e-6696d3969bdc"
-					(reference "C9")
+					(reference "C11")
 					(unit 1)
 				)

Commit message: Esquemático Aquabox III
Other:
- company: (none) -> INVENCTUS Soluções Tecnológicas
- title: (none) -> Interfaces
Changed lines of the file:
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@@
 	(generator_version "10.0")
 	(paper "A4")
+	(title_block
+		(title "Interfaces")
+		(date "2026-07-29")
+		(rev "1.0.0")
+		(company "INVENCTUS Soluções Tecnológicas")
+		(comment 1 "Eng. José Adriano")
+		(comment 2 "AQUABOX III")
+	)
 	(text "ENTER"
 		(exclude_from_sim no)

Commit message: Atualização
Connections:
- net TFT_BL is gone; now on net +3.3V: J10.3 (Pin_3)
Changed lines of the file:
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@@
+	)
+	(junction
+		(at 222.25 50.8)
+		(diameter 0)
+		(color 0 0 0 0)
 	)
 	(junction
@@
 	(wire
 		(pts
+			(xy 222.25 53.34) (xy 222.25 50.8)
+		)
+		(stroke
+			(width 0)
+			(type default)
+		)
+	)
+	(wire
+		(pts
 			(xy 134.62 144.78) (xy 134.62 148.59)
 		)
@@
 	(wire
 		(pts
+			(xy 234.95 53.34) (xy 222.25 53.34)
+		)
+		(stroke
+			(width 0)
+			(type default)
+		)
+	)
+	(wire
+		(pts
 			(xy 59.69 55.88) (xy 72.39 55.88)
 		)
@@
 		(pts
 			(xy 167.64 110.49) (xy 175.26 110.49)
-		)
-		(stroke
-			(width 0)
-			(type default)
-		)
-	)
-	(wire
-		(pts
-			(xy 226.06 53.34) (xy 234.95 53.34)
 		)
 		(stroke
@@
 		(effects
 			(font
-				(size 1.27 1.27)
-			)
-			(justify right)
-		)
-	)
-	(hierarchical_label "TFT_BL"
-		(shape input)
-		(at 226.06 53.34 180)
-		(effects
-			(font
