File: hardware/aquabox_final/aquabox_final.kicad_sch (KiCad schematic)
At the start: 0 parts

Commit message: Atualização
Changed lines of the file:
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@@
 	(sheet
 		(at 64.77 93.98)
-		(size 30.48 15.24)
+		(size 33.02 15.24)
 		(exclude_from_sim no)
 		(in_bom yes)
@@
 	)
 	(sheet
-		(at 193.04 93.98)
+		(at 191.77 110.49)
 		(size 31.75 15.24)
 		(exclude_from_sim no)
@@
 		)
 		(property "Sheetname" "RTC_SD"
-			(at 193.04 93.2684 0)
+			(at 191.77 109.7784 0)
 			(show_name no)
 			(do_not_autoplace no)
@@
 		)
 		(property "Sheetfile" "rtc_sd.kicad_sch"
-			(at 193.04 109.8046 0)
+			(at 191.77 126.3146 0)
 			(show_name no)
 			(do_not_autoplace no)
@@
 	)
 	(sheet
-		(at 128.27 52.07)
+		(at 135.89 68.58)
 		(size 33.02 72.39)
 		(exclude_from_sim no)
@@
 		)
 		(property "Sheetname" "ESP32_S3"
-			(at 128.27 51.3584 0)
+			(at 135.89 67.8684 0)
 			(show_name no)
 			(do_not_autoplace no)
@@
 		)
 		(property "Sheetfile" "esp32_s3.kicad_sch"
-			(at 128.27 125.0446 0)
+			(at 135.89 141.5546 0)
 			(show_name no)
 			(do_not_autoplace no)
@@
 	)
 	(sheet
-		(at 63.5 55.88)
-		(size 31.75 13.97)
+		(at 64.77 44.45)
+		(size 31.75 15.24)
 		(exclude_from_sim no)
 		(in_bom yes)
@@
 		)
 		(property "Sheetname" "Power"
-			(at 63.5 55.1684 0)
+			(at 64.77 43.7384 0)
 			(show_name no)
 			(do_not_autoplace no)
@@
 		)
 		(property "Sheetfile" "power.kicad_sch"
-			(at 63.5 70.4346 0)
+			(at 64.77 60.2746 0)
 			(show_name no)
 			(do_not_autoplace no)
@@
 	)
 	(sheet
-		(at 191.77 58.42)
+		(at 189.23 45.72)
 		(size 31.75 15.24)
 		(exclude_from_sim no)
@@
 		)
 		(property "Sheetname" "Solenoids_Bomba"
-			(at 191.77 57.7084 0)
+			(at 189.23 45.0084 0)
 			(show_name no)
 			(do_not_autoplace no)
@@
 		)
 		(property "Sheetfile" "solenoids.kicad_sch"
-			(at 191.77 74.2446 0)
-			(show_name no)
-			(do_not_autoplace no)
+			(at 189.23 61.5446 0)
+			(show_name no)
+			(do_not_autoplace no)

Commit message: Atualização
Other:
- sheet Power ports: added R_C, R_NO; removed none
- sheet Solenoids_Bomba ports: added R_C, R_NO; removed none
Changed lines of the file:
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@@
 		(comment 1 "Eng. José Adriano")
+	)
+	(wire
+		(pts
+			(xy 96.52 50.8) (xy 201.93 50.8)
+		)
+		(stroke
+			(width 0)
+			(type default)
+		)
+	)
+	(wire
+		(pts
+			(xy 96.52 48.26) (xy 201.93 48.26)
+		)
+		(stroke
+			(width 0)
+			(type default)
+		)
 	)
 	(sheet
@@
 			)
 		)
+		(pin "R_NO" input
+			(at 96.52 50.8 0)
+			(effects
+				(font
+					(size 1.27 1.27)
+				)
+				(justify right)
+			)
+		)
+		(pin "R_C" output
+			(at 96.52 48.26 0)
+			(effects
+				(font
+					(size 1.27 1.27)
+				)
+				(justify right)
+			)
+		)
 		(instances
 			(project "aquabox_final"
@@
 	)
 	(sheet
-		(at 189.23 45.72)
+		(at 201.93 44.45)
 		(size 31.75 15.24)
 		(exclude_from_sim no)
@@
 		)
 		(property "Sheetname" "Solenoids_Bomba"
-			(at 189.23 45.0084 0)
+			(at 201.93 43.7384 0)
 			(show_name no)
 			(do_not_autoplace no)
@@
 		)
 		(property "Sheetfile" "solenoids.kicad_sch"
-			(at 189.23 61.5446 0)
-			(show_name no)
-			(do_not_autoplace no)
-			(effects
-				(font
-					(size 1.27 1.27)
-				)
-				(justify left top)
-			)
-		)
+			(at 201.93 60.2746 0)
+			(show_name no)
+			(do_not_autoplace no)
+			(effects
+				(font
+					(size 1.27 1.27)
+				)
+				(justify left top)
+			)
+		)
+		(pin "R_C" input
+			(at 201.93 48.26 180)
+			(effects
+				(font
+					(size 1.27 1.27)
+				)
+				(justify left)
+			)
+		)
+		(pin "R_NO" output
+			(at 201.93 50.8 180)
+			(effects
+				(font
+					(size 1.27 1.27)
+				)
+				(justify left)
+			)
+		)

Commit message: Atualização
Other:
- sheet Solenoids_Bomba renamed Outputs
- added sheet Interfaces (Interfaces.kicad_sch)
Changed lines of the file:
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@@
 	)
 	(sheet
-		(at 64.77 93.98)
+		(at 64.77 74.93)
 		(size 33.02 15.24)
 		(exclude_from_sim no)
@@
 		)
 		(property "Sheetname" "Inputs"
-			(at 64.77 93.2684 0)
+			(at 64.77 74.2184 0)
 			(show_name no)
 			(do_not_autoplace no)
@@
 		)
 		(property "Sheetfile" "inputs.kicad_sch"
-			(at 64.77 109.8046 0)
+			(at 64.77 90.7546 0)
 			(show_name no)
 			(do_not_autoplace no)
@@
 	)
 	(sheet
+		(at 66.04 109.22)
+		(size 33.02 20.32)
+		(exclude_from_sim no)
+		(in_bom yes)
+		(on_board yes)
+		(dnp no)
+		(fields_autoplaced yes)
+		(stroke
+			(width 0.1524)
+			(type solid)
+		)
+		(fill
+			(color 0 0 0 0)
+		)
+		(property "Sheetname" "Interfaces"
+			(at 66.04 108.5084 0)
+			(show_name no)
+			(do_not_autoplace no)
+			(effects
+				(font
+					(size 1.27 1.27)
+				)
+				(justify left bottom)
+			)
+		)
+		(property "Sheetfile" "Interfaces.kicad_sch"
+			(at 66.04 130.1246 0)
+			(show_name no)
+			(do_not_autoplace no)
+			(effects
+				(font
+					(size 1.27 1.27)
+				)
+				(justify left top)
+			)
+		)
+		(instances
+			(project "aquabox_final"
+				(path "/c895ac8d-c639-4fea-ba83-739985d9c75e"
+					(page "7")
+				)
+			)
+		)
+	)
+	(sheet
 		(at 201.93 44.45)
 		(size 31.75 15.24)
@@
 			(color 0 0 0 0)
 		)
-		(property "Sheetname" "Solenoids_Bomba"
+		(property "Sheetname" "Outputs"
 			(at 201.93 43.7384 0)
 			(show_name no)

Commit message: Atualização
Other:
- removed sheet RTC_SD
- sheet ESP32_S3 ports: added BOMBA_ON_OFF, BTN_BACK, BTN_DOWN, BTN_ENTER, BTN_UP, FLOW_COUNTER, MAN_AUTO, RELAY_PUMP, S1_HIGH, S1_LOW, S2_HIGH, S2_LOW, S3_HIGH, S3_LOW, SD_CS, SOL_1, SOL_2, SOL_3, SPI_MOSI, SPI_SCK, TFT_BL, TFT_CS, TFT_DC, TFT_RST; removed none
- sheet Inputs ports: added FLOW_COUNTER, S1_HIGH, S1_LOW, S2_HIGH, S2_LOW, S3_HIGH, S3_LOW; removed none
- sheet Interfaces ports: added BOMBA_ON_OFF, BTN_BACK, BTN_DOWN, BTN_ENTER, BTN_UP, MAN_AUTO, SD_CS, SPI_MOSI, SPI_SCK, TFT_BL, TFT_CS, TFT_DC, TFT_RST; removed none
- sheet Outputs ports: added RELAY_PUMP, SOL_1, SOL_2, SOL_3; removed none

Commit message: Esquemático Aquabox III
Other:
- note added: "DIAGRAMA DE CONEXÃO ENTRE MÓDULOS"
Changed lines of the file:
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@@
 		(comment 1 "Eng. José Adriano")
+	)
+	(text "DIAGRAMA DE CONEXÃO ENTRE MÓDULOS"
+		(exclude_from_sim no)
+		(at 147.32 27.686 0)
+		(effects
+			(font
+				(size 1.27 1.27)
+			)
+		)
 	)
 	(wire

Commit message: Atualização
Other:
- sheet ESP32_S3 ports: added none; removed TFT_BL
- sheet Interfaces ports: added none; removed TFT_BL
Changed lines of the file:
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@@
-	(wire
-		(pts
-			(xy 91.44 105.41) (xy 140.97 105.41)
-		)
-		(stroke
-			(width 0)
-			(type default)
-		)
-	)
 	(wire
 		(pts
@@
 			)
 		)
-		(pin "TFT_BL" output
-			(at 140.97 105.41 180)
-			(effects
-				(font
-					(size 1.27 1.27)
-				)
-				(justify left)
-			)
-		)
 		(pin "S3_HIGH" input
 			(at 140.97 85.09 180)
@@
 			(effects
 				(font
-					(size 1.27 1.27)
-				)
-				(justify right)
-			)
-		)
-		(pin "TFT_BL" input
-			(at 91.44 105.41 0)
-			(effects
-				(font
