File: hardware/aquabox_final/esp32_s3.kicad_sch (KiCad schematic)
At the start: 16 parts, among them J3 TFT - 1.8{dblquote} SPI, SW1 BOMBA, SW2 MANUAL?AUTOMATICO, U2 ESP32-S3-DEVKITC-1-N16R8V

Commit message: Atualização
Parts:
- removed C3, C4, C5, C6, C7, C8: 100n, symbol Device:C
- removed J3: TFT - 1.8{dblquote} SPI, 68664-008LF:AMPHENOL_68664-008LF, symbol Conect_2x10:68664-008LF
- removed R4, R5, R6, R7, R8, R9: 10K, symbol Device:R
- removed SW1: BOMBA, symbol Switch:SW_SPST
- removed SW2: MANUAL?AUTOMATICO, symbol Switch:SW_SPST
Connections:
- net T1_HIGH renamed S1_HIGH
- net T1_LOW renamed S1_LOW
- net T2_HIGH renamed S2_HIGH
- net T2_LOW renamed S2_LOW
- net T3_HIGH renamed S3_HIGH
- net T3_LOW renamed S3_LOW
Other:
- moved on the sheet: U2

Commit message: Atualização
Changed lines of the file:
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@@
+	(wire
+		(pts
+			(xy 175.26 90.17) (xy 185.42 90.17)
+		)
+		(stroke
+			(width 0)
+			(type default)
+		)
+	)
 	(wire
 		(pts
@@
 	(wire
 		(pts
-			(xy 175.26 82.55) (xy 182.88 82.55)
-		)
-		(stroke
-			(width 0)
-			(type default)
-		)
-	)
-	(wire
-		(pts
 			(xy 121.92 85.09) (xy 129.54 85.09)
 		)
@@
 	(wire
 		(pts
-			(xy 175.26 90.17) (xy 182.88 90.17)
-		)
-		(stroke
-			(width 0)
-			(type default)
-		)
-	)
-	(wire
-		(pts
 			(xy 121.92 100.33) (xy 129.54 100.33)
 		)
@@
 	(wire
 		(pts
+			(xy 175.26 82.55) (xy 185.42 82.55)
+		)
+		(stroke
+			(width 0)
+			(type default)
+		)
+	)
+	(wire
+		(pts
 			(xy 121.92 105.41) (xy 129.54 105.41)
 		)
@@
 			(width 0)
 			(type default)
-		)
-	)
-	(global_label "BOMBA_ON_OFF"
-		(shape input)
-		(at 182.88 82.55 0)
-		(fields_autoplaced yes)
-		(effects
-			(font
-				(size 1.27 1.27)
-			)
-			(justify left)
-		)
-		(property "Intersheetrefs" "${INTERSHEET_REFS}"
-			(at 200.3796 82.55 0)
-			(hide yes)
-			(show_name no)
-			(do_not_autoplace no)
-			(effects
-				(font
-					(size 1.27 1.27)
-				)
-				(justify left)
-			)
-		)
-	)
-	(global_label "MAN_AUTO"
-		(shape input)
-		(at 182.88 90.17 0)
-		(fields_autoplaced yes)
-		(effects
-			(font
-				(size 1.27 1.27)
-			)
-			(justify left)
-		)
-		(property "Intersheetrefs" "${INTERSHEET_REFS}"
-			(at 195.7834 90.17 0)
-			(hide yes)
-			(show_name no)
-			(do_not_autoplace no)
-			(effects
-				(font
-					(size 1.27 1.27)
-				)
-				(justify left)
-			)
 		)
 	)
@@
 		)
 	)
+	(hierarchical_label "BOMBA_ON_OFF"
+		(shape input)
+		(at 185.42 82.55 0)
+		(effects
+			(font
+				(size 1.27 1.27)
+			)
+			(justify left)
+		)
+	)
 	(hierarchical_label "TFT_DC"
 		(shape output)
@@
 		)
 	)
+	(hierarchical_label "MAN_AUTO"
+		(shape input)
+		(at 185.42 90.17 0)
+		(effects
+			(font
+				(size 1.27 1.27)
+			)
+			(justify left)
+		)
+	)

Commit message: Atualização
Parts:
- added BT1: Battery_Cell, Battery:Battery_Panasonic_CR2032-HFN_Horizontal_CircularHoles, symbol Device:Battery_Cell
- added C3: 100n, symbol Device:C
- added R4, R5, R6: 4K7, symbol Device:R
- added U3: DS3231M, Package_SO:SOIC-16W_7.5x10.3mm_P1.27mm, symbol Timer_RTC:DS3231M
Connections:
- net +3.3V: now also R4.1, R5.1, R6.1, U3.2 (VCC); no longer U2.J1_1 (3V3), U2.J1_2 (3V3)
- net GND: now also BT1.2 (-), C3.2, U3.10 (GND), U3.11 (GND), U3.12 (GND), U3.13 (GND), U3.5 (GND), U3.6 (GND), U3.7 (GND), U3.8 (GND), U3.9 (GND)
- net I2C_SCL: now also R4.2, U3.16 (SCL)
- net I2C_SDA: now also R5.2, U3.15 (SDA)
- net +5V: now reaches U2.J1_21 (5V0)
- new net: BT1.1 (+), C3.1, U3.14 (VBAT)
- new net: R6.2, U3.3 (~{INT}/SQW)
- new net 3V3: U2.J1_1 (3V3), U2.J1_2 (3V3)
- no-connect marks 12 -> 15
Other:
- moved on the sheet: U2

Commit message: Atualização
Parts:
- added C4: 100n, symbol Device:C
Connections:
- net +3.3V: now also C4.1
- net GND: now also C4.2

Commit message: Atualização
Connections:
- net TFT_BL: no longer names the net of U2.J1_7 (GPIO7)
Changed lines of the file:
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@@
-	(wire
-		(pts
-			(xy 62.23 96.52) (xy 69.85 96.52)
-		)
-		(stroke
-			(width 0)
-			(type default)
-		)
-	)
 	(wire
 		(pts
@@
 		(effects
 			(font
-				(size 1.27 1.27)
-			)
-			(justify right)
-		)
-	)
-	(hierarchical_label "TFT_BL"
-		(shape output)
-		(at 62.23 96.52 180)
-		(effects
-			(font
